Commit message: moveit motion planning using ompl

File: robot_description/urdf/arm_robot_control.xacro (robot description, xacro)
@@ -1,6 +1,6 @@
 <?xml version="1.0"?>
 <robot xmlns:xacro="http://www.ros.org/wiki/xacro" name="arm_robot">
-    <xacro:property name="PI" value="3.14159"/>
     <ros2_control name="RobotSystem" type="system">
+        <xacro:property name="PI" value="3.14159"/>
         <hardware>
             <plugin>gazebo_ros2_control/GazeboSystem</plugin>
@@ -8,6 +8,6 @@
         <joint name="joint_1">
             <command_interface name="position">
-                <params name="min">-${PI/2}</params>
-                <params name="max">${PI/2}</params>
+            <param name="min">-${PI/2}</param>
+            <param name="max">${PI/2}</param>
             </command_interface>
             <state_interface name="position"/>
@@ -15,6 +15,6 @@
         <joint name="joint_2">
             <command_interface name="position">
-                <params name="min">-${PI/2}</params>
-                <params name="max">${PI/2}</params>
+            <param name="min">-${PI/2}</param>
+            <param name="max">${PI/2}</param>
             </command_interface>
             <state_interface name="position"/>
@@ -22,6 +22,6 @@
         <joint name="joint_3">
             <command_interface name="position">
-                <params name="min">-${PI/2}</params>
-                <params name="max">${PI/2}</params>
+            <param name="min">-${PI/2}</param>
+            <param name="max">${PI/2}</param>
             </command_interface>
             <state_interface name="position"/>
@@ -29,6 +29,6 @@
         <joint name="joint_4">
             <command_interface name="position">
-                <params name="min">-${PI/2}</params>
-                <params name="max">0.0</params>
+            <param name="min">-${PI/2}</param>
+            <param name="max">0.0</param>
             </command_interface>
             <state_interface name="position"/>
@@ -38,8 +38,7 @@
             <param name="multiplier">-1</param>
             <command_interface name="position">
-                <params name="min">0.0</params>
-                <params name="max">${PI/2}</params>
+            <param name="min">0.0</param>
+            <param name="max">${PI/2}</param>
             </command_interface>
-            <state_interface name="position"/>
         </joint>
     </ros2_control>

File: robot_description/urdf/arm_robot_gazebo.xacro (robot description, xacro)
@@ -1,4 +1,4 @@
 <?xml version="1.0"?>
-<robot xmlns:xacro="http://www.ros.org/wiki/xacro">
+<robot xmlns:xacro="http://www.ros.org/wiki/xacro" name="arm_robot">
     <gazebo>
         <plugin filename="libgazebo_ros2_control.so" name="gazebo_ros2_control">

File: robot_description/urdf/robot_des.urdf.xacro (robot description, xacro)
@@ -64,5 +64,5 @@
         <child link="base_plate"/>
         <axis xyz="0 0 1"/>
-        <origin rpy="0 0 0" xyz="0 0 0.307"/>
+        <origin xyz="0 0 0.307"/>
         <limit lower="-${PI/2}" upper="${PI/2}" effort="${effort}" velocity="${velocity}"/>
     </joint>
@@ -108,5 +108,5 @@
         <child link="horizontal_arm"/>
         <axis xyz="1 0 0"/>
-        <origin rpy="0 0 0" xyz="0 0 0.8"/>
+        <origin xyz="0 0 0.8"/>
         <limit lower="-${PI/2}" upper="${PI/2}" effort="${effort}" velocity="${velocity}"/>
     </joint>
@@ -129,7 +129,5 @@
         <parent link="horizontal_arm"/>
         <child link="claw_support"/>
-        <axis xyz="1 0 0"/>
-        <origin rpy="0 0 0" xyz="0 0.82 0"/>
-        <limit lower="-${PI/2}" upper="${PI/2}" effort="${effort}" velocity="${velocity}"/>
+        <origin xyz="0 0.82 0"/>
     </joint>
     <link name="gripper_right">
@@ -174,5 +172,5 @@
         <child link="gripper_left"/>
         <axis xyz="0 0 1"/>
-        <origin rpy="0 0 0" xyz="-0.22 0.13 -0.1"/>
+        <origin xyz="-0.22 0.13 -0.1"/>
         <limit lower="0.0" upper="${PI/2}" effort="${effort}" velocity="${velocity}"/>
         <mimic joint="joint_4" multiplier="-1"/>
